File: HW/VQFN-kicad-version/xyp-gpib.kicad_pcb (KiCad board)
At the start: 2 copper layers, 56.2 x 39.3 mm, 19 parts, among them J1 USB_B, U1 ATmega32U4-MU, Y1 Crystal_GND24

Commit message: October 2023 updates
- 488.2 support is enabled.
- fixed issue: Linux PCs show that Config 1 descriptor is not correct.
- Fixed read status byte, Clear and trigger assertion functions.
- Compatibility with R&S Visa is back - it got broken in a previous version. Read status byte, Clear and trigger did not work properly.
- I deleted 2 HW variants to avoid confusion. Right now there is one Eagle 6 version (mine) and a user contributed Kicad version included.
Routing:
- added copper zone on B.Cu, net GND
