File: HW/REV2/KicadV2/xyp-gpib.kicad_sch (KiCad schematic)
At the start: 26 parts, among them J1 USB_C_Receptacle_USB2.0, SW1 SW_Push, U1 ATmega32U4-MU, U2 USBLC6-2P6, Y1 CX2016DB16000D0WZRC1

Commit message: [FIX] Value of C5/C6 seems to be wrong
Signed-off-by: Silvano Cortesi <silvano.cortesi@hotmail.com>
Parts:
- C5, C6: value 8pF -> 18pF
Changed lines of the file:
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@@
 			)
 		)
-		(property "Value" "8pF"
+		(property "Value" "18pF"
 			(at 114.3 78.105 90)
 			(effects
@@
 			)
 		)
-		(property "Value" "8pF"
+		(property "Value" "18pF"
 			(at 114.3 63.2206 90)
 			(effects
